Commit message: 修正：老车模型使用固定云台兼容 TF

File: src/rm_description/urdf/rm_old_car_2026.urdf.xacro (robot description, xacro)
@@ -23,13 +23,12 @@
     </visual>
   </link>
-  <!-- The old car has no navigation gimbal. Keep a zero-yaw compatibility
-       joint so the existing gimbal_state_adapter and canonical TF chain can
-       be reused without changing frame ownership. -->
+  <!-- The old car has no navigation gimbal. Keep a fixed zero-yaw
+       compatibility frame so description-only validation can publish the full
+       TF chain without requiring a /joint_states source. -->
   <link name="gimbal_yaw_link"/>
-  <joint name="gimbal_yaw_joint" type="continuous">
+  <joint name="gimbal_yaw_joint" type="fixed">
     <parent link="base_link"/>
     <child link="gimbal_yaw_link"/>
     <origin xyz="0 0 0" rpy="0 0 0"/>
-    <axis xyz="0 0 1"/>
   </joint>
   <link name="lio_imu_link"/>

Commit message: 实验：接入老车左雷达点云 costmap 配置

File: src/rm_description/urdf/rm_old_car_2026.urdf.xacro (robot description, xacro)
@@ -45,4 +45,11 @@
     <origin xyz="0.15 0.14 0.24" rpy="0 0 0"/>
   </joint>
+  <link name="mid360_left_frame"/>
+  <joint name="gimbal_yaw_link_to_mid360_left_frame" type="fixed">
+    <parent link="gimbal_yaw_link"/>
+    <child link="mid360_left_frame"/>
+    <!-- Matches the current left driver frame_id and old-car placeholder. -->
+    <origin xyz="0.15 0.14 0.24" rpy="0 0 0"/>
+  </joint>
   <link name="base_imu_link"/>
   <joint name="base_link_to_base_imu_link" type="fixed">

Commit message: 修复外参

File: src/rm_description/urdf/rm_old_car_2026.urdf.xacro (robot description, xacro)
@@ -3,13 +3,28 @@
   <!--
     Old-car validation model only.
-    The lidar/IMU placeholder below is derived from the old 2026 URDF:
-      rm2026_navigation/src/robot_msgs/urdf/car.urdf.xacro
-      joint_laser_x = 0.15
-      joint_laser_y = 0.14
-      joint_laser_z = 0.24
-      rpy = 0 0 0
+    The old-car MID360 transform below uses the final 2026 measured L1
+    extrinsic from:
+      rm2026_navigation/src/robot_msgs/urdf/robot.urdf
+      rm2026_navigation/radar_multi_notice.md
+    Source measurement was left-handed with x forward, y right, z up:
+      L1 position: (193.5, -175.3, 210.2) mm
+      L1 normal:   (3.91, -3.91, 11.87)
+    Converted to ROS x-forward, y-left, z-up:
+      xyz=(0.1935, 0.1753, 0.2102)
+      rpy=(0.332345, 0.287549, 1.668370)
+    MID360 internal IMU to lidar offset from the 2026 FAST-LIO config:
+      imu->lidar xyz=(-0.011, -0.02329, 0.04412), rpy=(0, 0, 0)
     This file must not be used as 2027 robot calibration. It exists only for
     the experiment/old-car-2026-bringup validation branch.
   -->
+  <xacro:property name="old_car_l1_x" value="0.1935"/>
+  <xacro:property name="old_car_l1_y" value="0.1753"/>
+  <xacro:property name="old_car_l1_z" value="0.2102"/>
+  <xacro:property name="old_car_l1_roll" value="0.332345"/>
+  <xacro:property name="old_car_l1_pitch" value="0.287549"/>
+  <xacro:property name="old_car_l1_yaw" value="1.668370"/>
+  <xacro:property name="old_car_l1_imu_x" value="0.157178"/>
+  <xacro:property name="old_car_l1_imu_y" value="0.172624"/>
+  <xacro:property name="old_car_l1_imu_z" value="0.174374"/>
   <link name="base_link">
     <visual>
@@ -36,6 +51,8 @@
     <parent link="gimbal_yaw_link"/>
     <child link="lio_imu_link"/>
-    <!-- Old-car-only placeholder copied from the 2026 laser joint. -->
-    <origin xyz="0.15 0.14 0.24" rpy="0 0 0"/>
+    <!-- Selected MID360 internal IMU frame used by FAST-LIO body state. -->
+    <origin
+      xyz="${old_car_l1_imu_x} ${old_car_l1_imu_y} ${old_car_l1_imu_z}"
+      rpy="${old_car_l1_roll} ${old_car_l1_pitch} ${old_car_l1_yaw}"/>
   </joint>
   <link name="old_car_laser_link"/>
@@ -43,5 +60,7 @@
     <parent link="gimbal_yaw_link"/>
     <child link="old_car_laser_link"/>
-    <origin xyz="0.15 0.14 0.24" rpy="0 0 0"/>
+    <origin
+      xyz="${old_car_l1_x} ${old_car_l1_y} ${old_car_l1_z}"
+      rpy="${old_car_l1_roll} ${old_car_l1_pitch} ${old_car_l1_yaw}"/>
   </joint>
   <link name="mid360_left_frame"/>
@@ -49,6 +68,8 @@
     <parent link="gimbal_yaw_link"/>
     <child link="mid360_left_frame"/>
-    <!-- Matches the current left driver frame_id and old-car placeholder. -->
-    <origin xyz="0.15 0.14 0.24" rpy="0 0 0"/>
+    <!-- Matches the current left driver frame_id and measured L1 extrinsic. -->
+    <origin
+      xyz="${old_car_l1_x} ${old_car_l1_y} ${old_car_l1_z}"
+      rpy="${old_car_l1_roll} ${old_car_l1_pitch} ${old_car_l1_yaw}"/>
   </joint>
   <link name="base_imu_link"/>

Commit message: 功能：新增双雷达障碍点云融合边界

File: src/rm_description/urdf/rm_old_car_2026.urdf.xacro (robot description, xacro)
@@ -27,4 +27,12 @@
   <xacro:property name="old_car_l1_imu_y" value="0.172624"/>
   <xacro:property name="old_car_l1_imu_z" value="0.174374"/>
+  <!-- Provisional L2 values from the documented 180-degree XOY symmetry.
+       They require physical measurement before dual-lidar acceptance. -->
+  <xacro:property name="old_car_l2_x" value="-0.1935"/>
+  <xacro:property name="old_car_l2_y" value="-0.1753"/>
+  <xacro:property name="old_car_l2_z" value="0.2102"/>
+  <xacro:property name="old_car_l2_roll" value="0.332345"/>
+  <xacro:property name="old_car_l2_pitch" value="0.287549"/>
+  <xacro:property name="old_car_l2_yaw" value="-1.473223"/>
   <link name="base_link">
     <visual>
@@ -73,4 +81,12 @@
       rpy="${old_car_l1_roll} ${old_car_l1_pitch} ${old_car_l1_yaw}"/>
   </joint>
+  <link name="mid360_right_frame"/>
+  <joint name="gimbal_yaw_link_to_mid360_right_frame" type="fixed">
+    <parent link="gimbal_yaw_link"/>
+    <child link="mid360_right_frame"/>
+    <origin
+      xyz="${old_car_l2_x} ${old_car_l2_y} ${old_car_l2_z}"
+      rpy="${old_car_l2_roll} ${old_car_l2_pitch} ${old_car_l2_yaw}"/>
+  </joint>
   <link name="base_imu_link"/>
   <joint name="base_link_to_base_imu_link" type="fixed">
